File: V3/Hardware/REV A/Toy-Audio.sch (KiCad schematic (older format))
At the start: 26 parts, among them J1 CONN_01X02, J2 CONN_01X04, J3 CONN_01X03, J4 CONN_01X03, J5 CONN_01X04, U1 XC6206P332MR, U2 STM32F030F4P6, U3 W25Q32FVSIG, U4 TS4890, U5 MCP48FEB02-E/UN

Commit message: Improved Wake-up pin stability WKUP1. modiefied schematic files. Software V1 is compatible with hardware V2
Parts:
- added R5: 10k, MvdL:R0603, symbol RR
Connections:
- net GND: now also R5.2
- net at J3.2 (P2), R2.2: now also R5.1
Other:
- moved on the sheet: R2
Changed lines of the file:
@@
 $EndComp
 $Comp
-L VDD #PWR01
+L VDD #PWR9
 U 1 1 55C87E0C
 P 3750 1700
-F 0 "#PWR01" H 3750 1550 50  0001 C CNN
+F 0 "#PWR9" H 3750 1550 50  0001 C CNN
 F 1 "VDD" H 3750 1850 50  0000 C CNN
 F 2 "" H 3750 1700 60  0000 C CNN
@@
 $EndComp
 $Comp
-L VDD #PWR02
+L VDD #PWR13
 U 1 1 55D300D4
 P 4250 1700
-F 0 "#PWR02" H 4250 1550 50  0001 C CNN
+F 0 "#PWR13" H 4250 1550 50  0001 C CNN
 F 1 "VDD" H 4250 1850 50  0000 C CNN
 F 2 "" H 4250 1700 60  0000 C CNN
@@
 MISO1
 $Comp
-L VCC #PWR03
+L VCC #PWR6
 U 1 1 55DE7341
 P 2550 1700
-F 0 "#PWR03" H 2550 1550 50  0001 C CNN
+F 0 "#PWR6" H 2550 1550 50  0001 C CNN
 F 1 "VCC" H 2550 1850 50  0000 C CNN
 F 2 "" H 2550 1700 60  0000 C CNN
@@
 $EndComp
 $Comp
-L VDD #PWR04
+L VDD #PWR19
 U 1 1 55DE7A85
 P 6000 1650
-F 0 "#PWR04" H 6000 1500 50  0001 C CNN
+F 0 "#PWR19" H 6000 1500 50  0001 C CNN
 F 1 "VDD" H 6000 1800 50  0000 C CNN
 F 2 "" H 6000 1650 60  0000 C CNN
@@
 $EndComp
 $Comp
-L GND #PWR05
+L GND #PWR2
 U 1 1 55DEC140
 P 1500 4150
-F 0 "#PWR05" H 1500 3900 50  0001 C CNN
+F 0 "#PWR2" H 1500 3900 50  0001 C CNN
 F 1 "GND" H 1500 4000 50  0000 C CNN
 F 2 "" H 1500 4150 60  0000 C CNN
@@
 $EndComp
 $Comp
-L GND #PWR06
+L GND #PWR1
 U 1 1 55DEC4CC
 P 1500 2250
-F 0 "#PWR06" H 1500 2000 50  0001 C CNN
+F 0 "#PWR1" H 1500 2000 50  0001 C CNN
 F 1 "GND" H 1500 2100 50  0000 C CNN
 F 2 "" H 1500 2250 60  0000 C CNN
@@
 $EndComp
 $Comp
-L GND #PWR07
+L GND #PWR8
 U 1 1 55DEC686
 P 3150 2250
-F 0 "#PWR07" H 3150 2000 50  0001 C CNN
+F 0 "#PWR8" H 3150 2000 50  0001 C CNN
 F 1 "GND" H 3150 2100 50  0000 C CNN
 F 2 "" H 3150 2250 60  0000 C CNN
@@
 $EndComp
 $Comp
-L GND #PWR08
+L GND #PWR10
 U 1 1 55DEC763
 P 3750 2250
-F 0 "#PWR08" H 3750 2000 50  0001 C CNN
+F 0 "#PWR10" H 3750 2000 50  0001 C CNN
 F 1 "GND" H 3750 2100 50  0000 C CNN
 F 2 "" H 3750 2250 60  0000 C CNN
@@
 $EndComp
 $Comp
-L GND #PWR09
+L GND #PWR20
 U 1 1 55DEE40F
 P 6000 2250
-F 0 "#PWR09" H 6000 2000 50  0001 C CNN
+F 0 "#PWR20" H 6000 2000 50  0001 C CNN
 F 1 "GND" H 6000 2100 50  0000 C CNN
 F 2 "" H 6000 2250 60  0000 C CNN
@@
 $EndComp
 $Comp
-L GND #PWR010
+L GND #PWR14
 U 1 1 55DEE754
 P 4250 2250
-F 0 "#PWR010" H 4250 2000 50  0001 C CNN
+F 0 "#PWR14" H 4250 2000 50  0001 C CNN
 F 1 "GND" H 4250 2100 50  0000 C CNN
 F 2 "" H 4250 2250 60  0000 C CNN
@@
 $EndComp
 $Comp
-L GND #PWR011
+L GND #PWR33
 U 1 1 55EC5978
 P 10950 4250
-F 0 "#PWR011" H 10950 4000 50  0001 C CNN
+F 0 "#PWR33" H 10950 4000 50  0001 C CNN
 F 1 "GND" H 10950 4100 50  0000 C CNN
 F 2 "" H 10950 4250 60  0000 C CNN
@@
 MOSI1
 $Comp
-L GND #PWR012
+L GND #PWR23
 U 1 1 55ECAB8E
 P 7000 1700
-F 0 "#PWR012" H 7000 1450 50  0001 C CNN
+F 0 "#PWR23" H 7000 1450 50  0001 C CNN
 F 1 "GND" H 7000 1550 50  0000 C CNN
 F 2 "" H 7000 1700 60  0000 C CNN
@@
 nHOLD
 $Comp
-L VCC #PWR013
+L VCC #PWR4
 U 1 1 55EDF925
 P 1600 3700
-F 0 "#PWR013" H 1600 3550 50  0001 C CNN
+F 0 "#PWR4" H 1600 3550 50  0001 C CNN
 F 1 "VCC" H 1600 3850 50  0000 C CNN
 F 2 "" H 1600 3700 60  0000 C CNN
@@
 $EndComp
 $Comp
-L GND #PWR014
+L GND #PWR31
 U 1 1 55EDFECB
 P 10300 2100
-F 0 "#PWR014" H 10300 1850 50  0001 C CNN
+F 0 "#PWR31" H 10300 1850 50  0001 C CNN
 F 1 "GND" H 10300 1950 50  0000 C CNN
 F 2 "" H 10300 2100 60  0000 C CNN
@@
 $EndComp
 $Comp
-L VDD #PWR015
+L VDD #PWR30
 U 1 1 55EDFFBE
 P 10300 1500
-F 0 "#PWR015" H 10300 1350 50  0001 C CNN
+F 0 "#PWR30" H 10300 1350 50  0001 C CNN
 F 1 "VDD" H 10300 1650 50  0000 C CNN
 F 2 "" H 10300 1500 60  0000 C CNN
@@
 $EndComp
 $Comp
-L VDD #PWR016
+L VDD #PWR17
 U 1 1 55EF3935
 P 5000 1100
-F 0 "#PWR016" H 5000 950 50  0001 C CNN
+F 0 "#PWR17" H 5000 950 50  0001 C CNN
 F 1 "VDD" H 5000 1250 50  0000 C CNN
 F 2 "" H 5000 1100 60  0000 C CNN
@@
 nHOLD
 $Comp
-L GND #PWR017
+L GND #PWR7
 U 1 1 566EDE46
 P 2850 4150
-F 0 "#PWR017" H 2850 3900 50  0001 C CNN
+F 0 "#PWR7" H 2850 3900 50  0001 C CNN
 F 1 "GND" H 2850 4000 50  0000 C CNN
 F 2 "" H 2850 4150 60  0000 C CNN
@@
 SCL1
 $Comp
-L GND #PWR018
+L GND #PWR11
 U 1 1 566EE888
 P 3750 6200
-F 0 "#PWR018" H 3750 5950 50  0001 C CNN
+F 0 "#PWR11" H 3750 5950 50  0001 C CNN
 F 1 "GND" H 3750 6050 50  0000 C CNN
 F 2 "" H 3750 6200 60  0000 C CNN
@@
 L RR R2
 U 1 1 566EF481
-P 1600 5900
-F 0 "R2" V 1700 6100 50  0000 C CNN
-F 1 "470R" V 1700 5900 50  0000 C CNN
-F 2 "MvdL:R0603" H 1600 5900 60  0001 C CNN
-F 3 "" H 1600 5900 60  0000 C CNN
-	1    1600 5900
+P 1250 5900
+F 0 "R2" V 1350 6100 50  0000 C CNN
+F 1 "470R" V 1350 5900 50  0000 C CNN
+F 2 "MvdL:R0603" H 1250 5900 60  0001 C CNN
+F 3 "" H 1250 5900 60  0000 C CNN
+	1    1250 5900
 	0    -1   -1   0
 $EndComp
-Text Label 1000 5900 0    60   ~ 0
+Text Label 650  5900 0    60   ~ 0
 WKUP1
-Text Label 1000 6000 0    60   ~ 0
+Text Label 650  6000 0    60   ~ 0
 LED
 $Comp
-L GND #PWR019
+L GND #PWR5
 U 1 1 566EFA35
 P 2200 6200
-F 0 "#PWR019" H 2200 5950 50  0001 C CNN
+F 0 "#PWR5" H 2200 5950 50  0001 C CNN
 F 1 "GND" H 2200 6050 50  0000 C CNN
 F 2 "" H 2200 6200 60  0000 C CNN
@@
 $EndComp
 $Comp
-L VDD #PWR020
+L VDD #PWR12
 U 1 1 566F13F5
 P 3850 5750
-F 0 "#PWR020" H 3850 5600 50  0001 C CNN
+F 0 "#PWR12" H 3850 5600 50  0001 C CNN
 F 1 "VDD" H 3850 5900 50  0000 C CNN
 F 2 "" H 3850 5750 60  0000 C CNN
@@
 $EndComp
 $Comp
-L GND #PWR021
+L GND #PWR29
 U 1 1 566ED17C
 P 9300 4550
-F 0 "#PWR021" H 9300 4300 50  0001 C CNN
+F 0 "#PWR29" H 9300 4300 50  0001 C CNN
 F 1 "GND" H 9300 4400 50  0000 C CNN
 F 2 "" H 9300 4550 60  0000 C CNN
@@
 $EndComp
 $Comp
-L GND #PWR022
+L GND #PWR27
 U 1 1 566ED1A5
 P 8650 4550
-F 0 "#PWR022" H 8650 4300 50  0001 C CNN
+F 0 "#PWR27" H 8650 4300 50  0001 C CNN
 F 1 "GND" H 8650 4400 50  0000 C CNN
 F 2 "" H 8650 4550 60  0000 C CNN
@@
 	2200 5800 2200 6200
 Wire Wire Line
-	1800 5900 2250 5900
+	1450 5900 2250 5900
 Wire Wire Line
 	2150 6000 2250 6000
 Wire Wire Line
-	1000 5900 1350 5900
-Wire Wire Line
-	1000 6000 1700 6000
+	650  5900 1000 5900
+Wire Wire Line
+	650  6000 1700 6000
 Wire Wire Line
 	1500 2250 1500 2000
@@
 nMUTE
 $Comp
-L VCC #PWR023
+L VCC #PWR32
 U 1 1 55EE03DA
 P 10950 3750
-F 0 "#PWR023" H 10950 3600 50  0001 C CNN
+F 0 "#PWR32" H 10950 3600 50  0001 C CNN
 F 1 "VCC" H 10950 3900 50  0000 C CNN
 F 2 "" H 10950 3750 60  0000 C CNN
@@
 $EndComp
 $Comp
-L VCC #PWR024
+L VCC #PWR28
 U 1 1 566F4888
 P 9300 3400
-F 0 "#PWR024" H 9300 3250 50  0001 C CNN
+F 0 "#PWR28" H 9300 3250 50  0001 C CNN
 F 1 "VCC" H 9300 3550 50  0000 C CNN
 F 2 "" H 9300 3400 60  0000 C CNN
@@
 Text Notes 2350 3350 0    60   ~ 0
 Serial Interface
-Text Notes 1400 5550 0    60   ~ 0
+Text Notes 1050 5550 0    60   ~ 0
 Button and LED
 Text Notes 3350 5450 0    60   ~ 0
@@
 	5200 3850 5600 3850
 $Comp
-L VDD #PWR025
+L VDD #PWR21
 U 1 1 56749C9B
 P 6650 3450
-F 0 "#PWR025" H 6650 3300 50  0001 C CNN
+F 0 "#PWR21" H 6650 3300 50  0001 C CNN
 F 1 "VDD" H 6650 3600 50  0000 C CNN
 F 2 "" H 6650 3450 60  0000 C CNN
@@
 $EndComp
 $Comp
-L GND #PWR026
+L GND #PWR22
 U 1 1 56749CE8
 P 6650 4150
-F 0 "#PWR026" H 6650 3900 50  0001 C CNN
+F 0 "#PWR22" H 6650 3900 50  0001 C CNN
 F 1 "GND" H 6650 4000 50  0000 C CNN
 F 2 "" H 6650 4150 60  0000 C CNN
@@
 $EndComp
 $Comp
-L VDD #PWR027
+L VDD #PWR15
 U 1 1 5674AE1A
 P 4700 3500
-F 0 "#PWR027" H 4700 3350 50  0001 C CNN
+F 0 "#PWR15" H 4700 3350 50  0001 C CNN
 F 1 "VDD" H 4700 3650 50  0000 C CNN
 F 2 "" H 4700 3500 60  0000 C CNN
@@
 $EndComp
 $Comp
-L GND #PWR028
+L GND #PWR16
 U 1 1 5674AE20
 P 4700 4050
-F 0 "#PWR028" H 4700 3800 50  0001 C CNN
+F 0 "#PWR16" H 4700 3800 50  0001 C CNN
 F 1 "GND" H 4700 3900 50  0000 C CNN
 F 2 "" H 4700 4050 60  0000 C CNN
@@
 $EndComp
 $Comp
-L GND #PWR029
+L GND #PWR24
 U 1 1 5674B0BB
 P 7050 4150
-F 0 "#PWR029" H 7050 3900 50  0001 C CNN
+F 0 "#PWR24" H 7050 3900 50  0001 C CNN
 F 1 "GND" H 7050 4000 50  0000 C CNN
 F 2 "" H 7050 4150 60  0000 C CNN
@@
 DAC
 $Comp
-L VDD #PWR030
+L VDD #PWR25
 U 1 1 56754F3C
 P 8000 1050
-F 0 "#PWR030" H 8000 900 50  0001 C CNN
+F 0 "#PWR25" H 8000 900 50  0001 C CNN
 F 1 "VDD" H 8000 1200 50  0000 C CNN
 F 2 "" H 8000 1050 60  0000 C CNN
@@
 $EndComp
 $Comp
-L VDD #PWR031
+L VDD #PWR18
 U 1 1 567752BE
 P 5525 2900
-F 0 "#PWR031" H 5525 2750 50  0001 C CNN
+F 0 "#PWR18" H 5525 2750 50  0001 C CNN
 F 1 "VDD" H 5525 3050 50  0000 C CNN
 F 2 "" H 5525 2900 60  0000 C CNN
@@
 $EndComp
 $Comp
-L GND #PWR032
+L GND #PWR26
 U 1 1 56775664
 P 8300 4550
-F 0 "#PWR032" H 8300 4300 50  0001 C CNN
+F 0 "#PWR26" H 8300 4300 50  0001 C CNN
 F 1 "GND" H 8300 4400 50  0000 C CNN
 F 2 "" H 8300 4550 60  0000 C CNN
@@
 	8300 4000 8300 4050
 Connection ~ 8300 4000
+$Comp
+L RR R5
+U 1 1 56785CE0
+P 1500 6325
+F 0 "R5" H 1625 6450 50  0000 C CNN
+F 1 "10k" H 1650 6325 50  0000 C CNN
+F 2 "MvdL:R0603" H 1500 6325 60  0001 C CNN
+F 3 "" H 1500 6325 60  0000 C CNN
+	1    1500 6325
+	1    0    0    -1
+$EndComp
+$Comp
+L GND #PWR3
+U 1 1 56785EAB
+P 1500 6600
+F 0 "#PWR3" H 1500 6350 50  0001 C CNN
+F 1 "GND" H 1500 6450 50  0000 C CNN
+F 2 "" H 1500 6600 60  0000 C CNN
+F 3 "" H 1500 6600 60  0000 C CNN
+	1    1500 6600
+	1    0    0    -1
+$EndComp
+Wire Wire Line
+	1500 6525 1500 6600
+Wire Wire Line
+	1500 6075 1500 5900
+Connection ~ 1500 5900
 $EndSCHEMATC
