File: V1/REV A/Toy-Audio.sch (KiCad schematic (older format))
At the start: 18 parts, among them J1 CONN_2, J2 CONN_01X04, J3 CONN_01X10, Q1 Si2302DS, U1 XC6206P332MR, U2 STM32F030F4P6, U3 W25Q32FVSIG

Commit message: Added support for SPI FLASH power down function
Parts:
- U1: value XC6206P332MR -> XC6206P282MR
Other:
- note added: "4.5V (or 3V)"
- note added: "Do not place U1 when using 3V battery power\nbypass pin 2 and 3 with a 0 Ohm resistor"
- note removed: "3V"
- note removed: "Do not place U1 when using 3V battery power\nbypass pin 2 and 3"
- note removed: "Optional HPF with 4KHz cutoff to filter \nout the PWM base frequency"
Changed lines of the file:
@@
 Text Label 5450 4300 0    60   ~ 0
 nCS
-Text Notes 1250 4850 0    60   ~ 0
+Text Notes 900  4675 0    60   ~ 0
 Battery Power
 Text Label 1050 3750 0    60   ~ 0
@@
 P 3100 5100
 F 0 "U1" H 3200 5150 60  0000 C CNN
-F 1 "XC6206P332MR" H 3100 5450 60  0000 C CNN
+F 1 "XC6206P282MR" H 3100 5450 60  0000 C CNN
 F 2 "MvdL:SOT23" H 3100 5050 60  0001 C CNN
 F 3 "" H 3100 5050 60  0000 C CNN
@@
 Wire Wire Line
 	1400 3550 1600 3550
-Text Notes 9150 2500 0    60   ~ 0
-Optional HPF with 4KHz cutoff to filter \nout the PWM base frequency
 Text Notes 9500 4300 0    60   ~ 0
 d.n.p. = do not place
-Text Notes 1900 4850 0    60   ~ 0
-3V
+Text Notes 900  4775 0    60   ~ 0
+4.5V (or 3V)
 Wire Notes Line
 	2650 4850 2650 4600
@@
 	3550 4600 3550 4850
 Text Notes 2200 4450 0    60   ~ 0
-Do not place U1 when using 3V battery power\nbypass pin 2 and 3
+Do not place U1 when using 3V battery power\nbypass pin 2 and 3 with a 0 Ohm resistor
 Wire Notes Line
 	8875 4100 8875 4150

Commit message: added resistor between Speaker + and Vbat to improve stability during playback. (HW V1)
Parts:
- R3: value 0R -> d.n.p.
Connections:
- net +BATT: now reaches D1.A, J1.2 (PM)
- net USART1_CTS renamed WKUP1
Other:
- note added: "100k"
- note added: "10k"
- note added: "12R 0.5W"
- note added: "SP1 should be a 32 Ohm speaker. \nWhen using a 16 Ohm Speaker connect\nSP+ trough a 12 Ohm resistor to +BATT"
- note removed: "12k"

Commit message: Minimized HW REV A, merged programming Terminal menu into main code. the menu is entered when data is received on the serial interface.
Parts:
- C1: value 10u -> d.n.p.
- C10: value 10uF -> d.n.p.
- C5: value 100n -> d.n.p.
- SP1: value 16Ohm -> 8Ohm
Connections:
- net +BATT: now also C8.1, R3.1, SP1.2
Other:
- note added: "or 16Ohm\nor 32Ohm"
- note removed: "12R 0.5W"
- note removed: "SP1 should be a 32 Ohm speaker. \nWhen using a 16 Ohm Speaker connect\nSP+ trough a 12 Ohm resistor to +BATT"
Changed lines of the file:
@@
 Sheet 1 1
 Title "Toy Audio V1"
-Date "5 aug 2015"
+Date "2016-01-06"
 Rev "A"
 Comp "Maurits van de Lande (maurits@vandelande.com)"
@@
 P 10000 3600
 F 0 "SP1" H 9800 3900 60  0000 C CNN
-F 1 "16Ohm" H 9800 3300 60  0000 C CNN
+F 1 "8Ohm" H 9800 3300 60  0000 C CNN
 F 2 "MvdL:JST-PH-2P-DUAL" H 10000 3600 60  0001 C CNN
 F 3 "~" H 10000 3600 60  0000 C CNN
@@
 P 10350 3600
 F 0 "C10" H 10350 3700 40  0000 L CNN
-F 1 "10uF" H 10356 3515 40  0000 L CNN
+F 1 "d.n.p." H 10356 3515 40  0000 L CNN
 F 2 "MvdL:C0603" H 10388 3450 30  0001 C CNN
 F 3 "~" H 10350 3600 60  0000 C CNN
@@
 P 2450 2000
 F 0 "C1" H 2450 2100 40  0000 L CNN
-F 1 "10u" H 2456 1915 40  0000 L CNN
+F 1 "d.n.p." H 2456 1915 40  0000 L CNN
 F 2 "MvdL:C0603" H 2488 1850 30  0001 C CNN
 F 3 "" H 2450 2000 60  0000 C CNN
@@
 P 3150 1900
 F 0 "C5" V 3200 1750 40  0000 L CNN
-F 1 "100n" V 3300 1850 40  0000 L CNN
+F 1 "d.n.p." V 3300 1850 40  0000 L CNN
 F 2 "MvdL:C0603" H 3188 1750 30  0001 C CNN
 F 3 "" H 3150 1900 60  0000 C CNN
@@
 	1    0    0    -1
 $EndComp
-Text Notes 9675 2850 0    60   ~ 0
-12R 0.5W
-Text Notes 8925 2325 0    60   ~ 0
-SP1 should be a 32 Ohm speaker. \nWhen using a 16 Ohm Speaker connect\nSP+ trough a 12 Ohm resistor to +BATT
 Text Notes 6500 2150 1    60   ~ 0
 10k
@@
 	9550 3500 9650 3500
 Wire Wire Line
-	9550 3500 9550 3400
+	9550 2650 9550 3500
 Wire Wire Line
 	9550 3400 9200 3400
@@
 	1575 4950 1575 5150
 Connection ~ 1575 5150
-Wire Notes Line
-	9550 2650 9550 2700
-Wire Notes Line
-	9550 2700 9600 2725
-Wire Notes Line
-	9600 2725 9500 2750
-Wire Notes Line
-	9500 2750 9600 2775
-Wire Notes Line
-	9600 2775 9500 2800
-Wire Notes Line
-	9500 2800 9600 2825
-Wire Notes Line
-	9600 2825 9500 2850
-Wire Notes Line
-	9500 2850 9600 2875
-Wire Notes Line
-	9600 2875 9500 2900
-Wire Notes Line
-	9500 2900 9600 2925
-Wire Notes Line
-	9600 2925 9550 2950
-Wire Notes Line
-	9550 2950 9550 3400
 Connection ~ 9550 3400
 Wire Notes Line
@@
 	1    0    0    -1
 $EndComp
+Wire Notes Line
+	9050 2925 9350 3300
+Wire Notes Line
+	9050 3300 9350 2925
+Text Notes 9550 4150 0    60   ~ 0
+or 16Ohm\nor 32Ohm
 $EndSCHEMATC
